File: kicad/key_matrix.kicad_sch (KiCad schematic)
At the start: 73 parts, among them SW1 SW_Push, SW10 SW_Push, SW11 SW_Push, SW12 SW_Push, SW13 SW_Push, SW14 SW_Push, SW15 SW_Push, SW16 SW_Push, SW17 SW_Push, SW18 SW_Push, SW19 SW_Push, SW2 SW_Push, SW20 SW_Push, SW21 SW_Push, SW22 SW_Push, SW23 SW_Push, SW24 SW_Push, SW25 SW_Push, SW26 SW_Push, SW27 SW_Push, SW28 SW_Push, SW29 SW_Push, SW3 SW_Push, SW30 SW_Push, SW31 SW_Push, SW32 SW_Push, SW33 SW_Push, SW34 SW_Push, SW35 SW_Push, SW36 Rotary_Encoder_Switch, SW4 SW_Push, SW5 SW_Push, SW6 SW_Push, SW7 SW_Push, SW8 SW_Push, SW9 SW_Push

Commit message: edited PCB
Parts:
- removed C18, C19: 100nF, Capacitor_SMD:C_0402_1005Metric, symbol Device:C
- removed D1, D10, D11, D12, D13, D14, D15, D16, D17, D18, D19, D2, D20, D21, D22, D23, D24, D25, D26, D27, D28, D29, D3, D30, D31, D32, D33, D34, D35, D4, D5, D6, D7, D8, D9: 1N4148W, Diode_SMD:D_SOD-123, symbol Diode:1N4148
- removed SW1, SW10, SW11, SW12, SW13, SW14, SW15, SW16, SW17, SW18, SW19, SW2, SW20, SW21, SW22, SW23, SW24, SW25, SW26, SW27, SW28, SW29, SW3, SW30, SW4, SW5, SW6, SW7, SW8, SW9: SW_Push, MX_hotswap_alps:MX-Hotswap-Alps-1U, symbol Switch:SW_Push
- removed SW31, SW34: SW_Push, MX_hotswap_alps:MX-Hotswap-Alps-1.25U, symbol Switch:SW_Push
- removed SW32, SW33: SW_Push, MX_hotswap_alps:MX-Hotswap-Alps-2U, symbol Switch:SW_Push
- removed SW35: SW_Push, MX_Alps_Hybrid:MX-Alps-Hybrid-1U, symbol Switch:SW_Push
- removed SW36: Rotary_Encoder_Switch, modified_footprints:RotaryEncoder_EC11_no_mp, symbol LeChiffre-rescue:Rotary_Encoder_Switch-Device
- added D1, D10, D11, D12, D13, D14, D15, D16, D17, D18, D19, D2, D20, D21, D22, D222, D23, D24, D25, D26, D27, D28, D29, D3, D30, D31, D32, D33, D34, D35, D36, D37, D38, D39, D4, D40, D41, D42, D43, D44, D45, D452, D46, D47, D48, D49, D5, D50, D51, D512, D52, D53, D54, D55, D56, D57, D58, D582, D59, D6, D60, D61, D62, D63, D64, D65, D66, D67, D68, D69, D7, D70, D71, D72, D73, D74, D75, D76, D77, D78, D79, D8, D80, D81, D812, D82, D83, D84, D85, D86, D87, D88, D89, D9, D90, D91: D_Small, Diode_SMD:D_SOD-123, symbol Device:D_Small
- added MX1, MX10, MX11, MX12, MX13, MX14, MX15, MX16, MX17, MX18, MX19, MX2, MX20, MX21, MX22, MX221, MX222, MX23, MX24, MX25, MX26, MX27, MX28, MX29, MX3, MX30, MX31, MX32, MX33, MX34, MX35, MX36, MX37, MX38, MX39, MX4, MX40, MX41, MX42, MX43, MX44, MX45, MX451, MX452, MX46, MX47, MX48, MX49, MX5, MX50, MX51, MX511, MX512, MX52, MX53, MX54, MX55, MX56, MX57, MX58, MX581, MX582, MX59, MX6, MX60, MX61, MX62, MX63, MX64, MX65, MX66, MX67, MX68, MX69, MX7, MX70, MX71, MX72, MX73, MX74, MX75, MX76, MX761, MX762, MX77, MX78, MX79, MX8, MX80, MX81, MX811, MX812, MX82, MX83, MX86, MX87, MX88, MX89, MX9, MX90: MX_SW_HS, PCM_marbastlib-mx:SW_MX_HS_1u, symbol PCM_marbastlib-mx:MX_SW_HS
- added MX84, MX85: MX_SW_HS, PCM_marbastlib-mx:SW_MX_HS_1.5u, symbol PCM_marbastlib-mx:MX_SW_HS
- added S1, S2, S3, S4, S5: MX_stab, PCM_marbastlib-mx:STAB_MX_P_2u, symbol PCM_marbastlib-mx:MX_stab
- added S6: MX_stab, PCM_marbastlib-mx:STAB_MX_P_4u, symbol PCM_marbastlib-mx:MX_stab
- added S7: MX_stab, PCM_marbastlib-mx:STAB_MX_P_2.75u, symbol PCM_marbastlib-mx:MX_stab
- added S8: MX_stab, PCM_marbastlib-mx:STAB_MX_P_2.25u, symbol PCM_marbastlib-mx:MX_stab
Connections:
- net col0: now also MX1.1, MX16.1, MX31.1, MX45.1, MX451.1, MX452.1, MX72.1, MX83.1
- net col1: now also MX17.1, MX2.1, MX32.1, MX46.1, MX60.1, MX73.1, MX84.1
- net col2: now also MX18.1, MX3.1, MX33.1, MX47.1, MX61.1, MX74.1
- net col3: now also MX19.1, MX34.1, MX4.1, MX48.1, MX62.1, MX75.1, MX85.1
- net col4: now also MX20.1, MX35.1, MX49.1, MX5.1, MX63.1
- net col5: now also MX21.1, MX36.1, MX50.1, MX6.1, MX64.1
- net col6: now also MX22.1, MX221.1, MX222.1, MX51.1, MX511.1, MX512.1, MX7.1, MX76.1, MX761.1
- net col7: now also MX23.1, MX37.1, MX52.1, MX65.1, MX762.1, MX8.1
- net col8: now also MX24.1, MX38.1, MX53.1, MX66.1, MX9.1
- net col9: now also MX10.1, MX25.1, MX39.1, MX54.1, MX67.1, MX77.1, MX86.1
- net row0: now also D1.1 (K), D10.1 (K), D11.1 (K), D12.1 (K), D13.1 (K), D14.1 (K), D15.1 (K), D2.1 (K), D3.1 (K), D4.1 (K), D5.1 (K), D6.1 (K), D7.1 (K), D8.1 (K), D9.1 (K)
- net row1: now also D16.1 (K), D17.1 (K), D18.1 (K), D19.1 (K), D20.1 (K), D21.1 (K), D22.1 (K), D23.1 (K), D24.1 (K), D25.1 (K), D26.1 (K), D27.1 (K), D28.1 (K), D29.1 (K), D30.1 (K)
- net row2: now also D222.1 (K), D31.1 (K), D32.1 (K), D33.1 (K), D34.1 (K), D35.1 (K), D36.1 (K), D37.1 (K), D38.1 (K), D39.1 (K), D40.1 (K), D41.1 (K), D42.1 (K), D43.1 (K), D44.1 (K)
- net row3: now also D45.1 (K), D46.1 (K), D47.1 (K), D48.1 (K), D49.1 (K), D50.1 (K), D51.1 (K), D52.1 (K), D53.1 (K), D54.1 (K), D55.1 (K), D56.1 (K), D57.1 (K), D58.1 (K), D59.1 (K)
- new net: D50.2 (A), MX50.2
- new net: D25.2 (A), MX25.2
- new net: D13.2 (A), MX13.2
- new net: D74.2 (A), MX74.2
- new net: D44.2 (A), MX44.2
- new net: D55.2 (A), MX55.2
- new net: D75.2 (A), MX75.2
- new net: D51.2 (A), MX51.2, MX511.2
- new net: D49.2 (A), MX49.2
- new net: D14.2 (A), MX14.2
- new net: D81.2 (A), MX81.2, MX811.2
- new net: D66.2 (A), MX66.2
- new net: D67.2 (A), MX67.2
- new net: D222.2 (A), MX222.2
- new net: D70.2 (A), MX70.2
- new net: D61.2 (A), MX61.2
- new net: D57.2 (A), MX57.2
- new net: D27.2 (A), MX27.2
- new net: D17.2 (A), MX17.2
- new net: D62.2 (A), MX62.2
- new net: D512.2 (A), MX512.2
- new net: D1.2 (A), MX1.2
- new net: D43.2 (A), MX43.2
- new net: D28.2 (A), MX28.2
- new net: D72.2 (A), MX72.2
- new net: D4.2 (A), MX4.2
- new net: D48.2 (A), MX48.2
- new net: D59.2 (A), MX59.2
- new net: D31.2 (A), MX31.2
- new net: D58.2 (A), MX58.2, MX581.2
- new net: D87.2 (A), MX87.2
- new net: D452.2 (A), MX452.2
- new net: D3.2 (A), MX3.2
- new net: D29.2 (A), MX29.2
- new net: D22.2 (A), MX22.2, MX221.2
- new net: D42.2 (A), MX42.2
- new net: D78.2 (A), MX78.2
- new net: D6.2 (A), MX6.2
- new net: D38.2 (A), MX38.2
- new net: D24.2 (A), MX24.2
- new net: D63.2 (A), MX63.2
- new net: D71.2 (A), MX71.2
- new net: D32.2 (A), MX32.2
- new net: D73.2 (A), MX73.2
- new net: D85.2 (A), MX85.2
- new net: D46.2 (A), MX46.2
- new net: D45.2 (A), MX45.2, MX451.2
- new net: D35.2 (A), MX35.2
- new net: D11.2 (A), MX11.2
- new net: D41.2 (A), MX41.2
- new net: D64.2 (A), MX64.2
- new net: D83.2 (A), MX83.2
- new net: D812.2 (A), MX812.2
- new net: D8.2 (A), MX8.2
- new net: D30.2 (A), MX30.2
- new net: D79.2 (A), MX79.2
- new net: D86.2 (A), MX86.2
- new net: D88.2 (A), MX88.2
- new net: D54.2 (A), MX54.2
- new net: D69.2 (A), MX69.2
- new net: D89.2 (A), MX89.2
- new net: D33.2 (A), MX33.2
- new net: D84.2 (A), MX84.2
- new net: D56.2 (A), MX56.2
- new net: D37.2 (A), MX37.2
- new net: D9.2 (A), MX9.2
- new net: D76.2 (A), MX76.2, MX761.2
- new net: D10.2 (A), MX10.2
- new net: D12.2 (A), MX12.2
- new net: D68.2 (A), MX68.2
- new net: D39.2 (A), MX39.2
- new net: D2.2 (A), MX2.2
- new net: D18.2 (A), MX18.2
- new net: D53.2 (A), MX53.2
- new net: D34.2 (A), MX34.2
- new net: D21.2 (A), MX21.2
- new net: D582.2 (A), MX582.2
- new net: D16.2 (A), MX16.2
- new net: D26.2 (A), MX26.2
- new net: D82.2 (A), MX82.2
- new net: D52.2 (A), MX52.2
- new net: D91.2 (A), MX762.2
- new net: D15.2 (A), MX15.2
- new net: D40.2 (A), MX40.2
- new net: D36.2 (A), MX36.2
- new net: D20.2 (A), MX20.2
- new net: D5.2 (A), MX5.2
- new net: D19.2 (A), MX19.2
- new net: D77.2 (A), MX77.2
- new net: D65.2 (A), MX65.2
- new net: D90.2 (A), MX90.2
- new net: D47.2 (A), MX47.2
- new net: D80.2 (A), MX80.2
- new net: D7.2 (A), MX7.2
- new net: D23.2 (A), MX23.2
- new net: D60.2 (A), MX60.2
- new net col10: MX11.1, MX26.1, MX40.1, MX55.1, MX68.1, MX78.1, MX87.1
- new net col11: MX12.1, MX27.1, MX41.1, MX56.1, MX69.1, MX79.1, MX88.1
- new net col12: MX13.1, MX28.1, MX42.1, MX57.1, MX70.1, MX80.1, MX89.1
- new net col13: MX14.1, MX29.1, MX43.1, MX58.1, MX581.1, MX582.1, MX81.1, MX811.1, MX812.1
- new net col14: MX15.1, MX30.1, MX44.1, MX59.1, MX71.1, MX82.1, MX90.1
- new net row4: D452.1 (K), D512.1 (K), D582.1 (K), D60.1 (K), D61.1 (K), D62.1 (K), D63.1 (K), D64.1 (K), D65.1 (K), D66.1 (K), D67.1 (K), D68.1 (K), D69.1 (K), D70.1 (K), D71.1 (K)
- new net row5: D72.1 (K), D73.1 (K), D74.1 (K), D75.1 (K), D76.1 (K), D77.1 (K), D78.1 (K), D79.1 (K), D80.1 (K), D81.1 (K), D82.1 (K), D91.1 (K)
- new net row6: D812.1 (K), D83.1 (K), D84.1 (K), D85.1 (K), D86.1 (K), D87.1 (K), D88.1 (K), D89.1 (K), D90.1 (K)
Other:
- company: sporkus -> jlw
- title: Hotswap Chiffre -> typomatrix
